File: MCL65+/PCBA/MCL65+.kicad_pcb (KiCad board)
At the start: 2 copper layers, 72.6 x 64.1 mm, 6 parts, among them U1 6502, U2 74HC14, U3 74LS573, U4 74LS573, U5 Teensy4.1

Commit message: modifications for PET 2001N
Other:
- net class Default removed
